File: ccnor_stm32_v24-sync.brd (EAGLE design)
At the start: 74.6 x 100 mm, 215 parts, among them J1 M02PT, J2 M02, Q10 WSP4406, Q11 NCE3018AS, Q12 NCE3018AS, Q13 WSP4406, Q16 2N7002P, Q2 WSP4406, Q3 WSP4406, Q7 IRLB8314PBF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

Commit message: Minor fixes/changes for cleanup
Minor fixes/changes for cleanup
Parts:
- moved F5 0.16 mm to (19.5, 3.02)
Other:
- board text added: "F1/3/5"
- board text added: "F2/4/6"
- board text removed: "0"
- board text removed: "F1/3"
- board text removed: "F2/4"
- board text removed: "Q4"
- board text removed: "R23"
- board text removed: "R36"
Changed lines of the file:
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@@
 <text x="34.29" y="96.67875" size="1.016" layer="22" font="vector" ratio="18" rot="MR90">GND</text>
 <text x="39.21125" y="96.67875" size="1.016" layer="22" font="vector" ratio="18" rot="MR90">VB</text>
-<text x="23.33625" y="69.5325" size="0.6096" layer="21" font="vector" ratio="18">0</text>
 <wire x1="0" y1="99" x2="0" y2="1" width="0" layer="20"/>
 <wire x1="34.29" y1="17.78" x2="34.29" y2="10.31875" width="0" layer="20"/>
@@
 <text x="6.19125" y="6.19125" size="0.6096" layer="21" font="vector" ratio="20" rot="R90">R37</text>
 <text x="6.19125" y="4.445" size="0.6096" layer="21" font="vector" ratio="20" rot="R90">R39</text>
-<text x="17.62125" y="4.92125" size="0.6096" layer="21" font="vector" ratio="20">F1/3</text>
-<text x="27.6225" y="1.984375" size="0.6096" layer="21" font="vector" ratio="20" rot="R90">Q1</text>
-<text x="26.82875" y="1.031875" size="0.6096" layer="21" font="vector" ratio="20">R23</text>
+<text x="18.415" y="0.635" size="0.6096" layer="21" font="vector" ratio="20">F1/3/5</text>
 <text x="26.51125" y="7.14375" size="0.6096" layer="21" font="vector" ratio="20" rot="R90">R72</text>
 <text x="24.28875" y="9.36625" size="0.6096" layer="21" font="vector" ratio="20">LED7</text>
@@
 <text x="24.92375" y="20.6375" size="0.6096" layer="21" font="vector" ratio="20">S1</text>
 <text x="48.73625" y="20.6375" size="0.6096" layer="21" font="vector" ratio="20">S2</text>
-<text x="46.355" y="1.11125" size="0.6096" layer="21" font="vector" ratio="20">R36</text>
-<text x="48.41875" y="5.55625" size="0.6096" layer="21" font="vector" ratio="20" rot="R90">Q4</text>
-<text x="54.76875" y="4.92125" size="0.6096" layer="21" font="vector" ratio="20">F2/4</text>
+<text x="53.0225" y="0.635" size="0.6096" layer="21" font="vector" ratio="20">F2/4/6</text>
 <text x="69.05625" y="4.445" size="0.6096" layer="21" font="vector" ratio="20" rot="R90">R40</text>
 <text x="69.05625" y="6.19125" size="0.6096" layer="21" font="vector" ratio="20" rot="R90">R38</text>
@@
 <element name="L5" library="custom" package="INDUCTOR_10A_8.2MMX21MM" value="60u" x="12.065" y="89.37625" rot="MR90"/>
 <element name="L6" library="custom" package="INDUCTOR_10A_8.2MMX21MM" value="60u" x="62.5475" y="89.37625" rot="MR270"/>
-<element name="F5" library="custom" package="2920" value="PTC2920" x="19.52625" y="3.175" rot="R180"/>
+<element name="F5" library="custom" package="2920" value="PTC2920" x="19.52625" y="3.01625" rot="R180"/>
 <element name="F6" library="custom" package="2920" value="PTC2920" x="55.08625" y="3.01625"/>
 <element name="U5" library="custom" package="SOT23-6" value="JW5052C" x="38.89375" y="84.7725"/>
@@
 <wire x1="11.4275" y1="4.7775" x2="11.43" y2="4.78" width="0.254" layer="1"/>
 <contactref element="F1" pad="2"/>
-<wire x1="15.5575" y1="3.175" x2="16.22625" y2="3.175" width="1.27" layer="1"/>
+<wire x1="15.5575" y1="3.175" x2="16.22625" y2="3.01625" width="1.27" layer="1"/>
 <contactref element="R54" pad="2"/>
-<wire x1="16.22625" y1="3.175" x2="16.2325" y2="3.175" width="1.27" layer="1"/>
+<wire x1="16.22625" y1="3.01625" x2="16.2325" y2="3.175" width="1.27" layer="1"/>
 <wire x1="17.765" y1="7.3025" x2="11.90625" y2="7.3025" width="0.254" layer="16"/>
 <wire x1="11.90625" y1="7.3025" x2="11.43" y2="7.77875" width="0.254" layer="16"/>
@@
 <wire x1="19.837" y1="2.8575" x2="20.6375" y2="2.8575" width="0.254" layer="1"/>
 <contactref element="F5" pad="A"/>
-<wire x1="22.82625" y1="3.175" x2="21.74875" y2="3.175" width="0.254" layer="1"/>
+<wire x1="22.82625" y1="3.01625" x2="21.74875" y2="3.175" width="0.254" layer="1"/>
 <wire x1="21.74875" y1="3.175" x2="21.43125" y2="2.8575" width="0.254" layer="1"/>
 </signal>
